File: senior_design/rc_ttt_remote/remote_pcb/remote_pcb.kicad_sch (KiCad schematic)
At the start: 13 parts, among them J1 Conn_02x01, SW1 SW_DIP_x01, SW2 SW_DIP_x01, SW3 SW_DIP_x01, SW4 SW_DIP_x01, SW5 SW_DIP_x01, SW6 SW_DIP_x01, U1 ESP32-DEVKIT-V1

Commit message: updated kicad files for remote
Parts:
- removed U1: ESP32-DEVKIT-V1, ESP32-DEVKIT-V1:MODULE_ESP32_DEVKIT_V1, symbol esp32-wroom:ESP32-DEVKIT-V1
- added D3: DB, LED_THT:LED_D3.0mm, symbol Device:LED
- added J2: PWR_TEST, Connector_PinHeader_2.54mm:PinHeader_1x02_P2.54mm_Vertical, symbol Connector_Generic:Conn_02x01
- added J3: PIN_TEST, Connector_PinHeader_2.54mm:PinHeader_1x02_P2.54mm_Vertical, symbol Connector_Generic:Conn_02x01
- added R3: 1K, Resistor_THT:R_Axial_DIN0204_L3.6mm_D1.6mm_P7.62mm_Horizontal, symbol Device:R
- added U2: ESP32-DEVKIT-V1, esp32_fp:MODULE_ESP32_DEVKIT_V1, symbol esp32-wroom:ESP32-DEVKIT-V1
- D1: value LED -> FW; footprint (none) -> LED_THT:LED_D3.0mm
- D2: value LED -> FB; footprint (none) -> LED_THT:LED_D3.0mm
- J1: value Conn_02x01 -> PWR; footprint (none) -> Connector_PinHeader_2.54mm:PinHeader_1x02_P2.54mm_Vertical
- R1, R2: footprint (none) -> Resistor_THT:R_Axial_DIN0204_L3.6mm_D1.6mm_P7.62mm_Horizontal
- S1: footprint EG1218:SW_EG1218 -> esp32_fp:SW_EG1218
- SW1: value SW_DIP_x01 -> LF; footprint (none) -> Button_Switch_THT:SW_PUSH-12mm
- SW2: value SW_DIP_x01 -> LB; footprint (none) -> Button_Switch_THT:SW_PUSH-12mm
- SW3: value SW_DIP_x01 -> FW; footprint (none) -> Button_Switch_THT:SW_PUSH-12mm
- SW4: value SW_DIP_x01 -> RF; footprint (none) -> Button_Switch_THT:SW_PUSH-12mm
- SW5: value SW_DIP_x01 -> RB; footprint (none) -> Button_Switch_THT:SW_PUSH-12mm
- SW6: value SW_DIP_x01 -> FB; footprint (none) -> Button_Switch_THT:SW_PUSH-12mm
Connections:
- net +3.3V: now also J2.1 (Pin_1)
- net GND: now also D3.1 (K), J2.2 (Pin_2), J3.2 (Pin_2), U2.2 (GND), U2.29 (GND)
- net at R1.2: now also U2.9 (D18)
- net at SW4.2: now also U2.27 (D12)
- net at SW1.2: now also U2.3 (D15)
- net at SW6.2: now also U2.26 (D14)
- net at SW3.2: now also U2.8 (D5)
- net at R2.2: now also U2.23 (D25)
- net at SW5.2: now also U2.28 (D13)
- net at S1.2: now also U2.30 (VIN)
- net at SW2.2: now also U2.5 (D4)
- new net: J3.1 (Pin_1), U2.11 (D21)
- new net: R3.2, U2.10 (D19)
- new net: D3.2 (A), R3.1
- no-connect marks 20 -> 18
